Commit message: moveit完成

File: src/arm_description/urdf/arm.xacro (robot description, xacro)
@@ -21,5 +21,5 @@
       <origin xyz="0 0 -0.005" rpy="0 0 0"/>
       <geometry>
-        <box size="0.08 0.08 0.01"/>
+        <box size="0.09 0.09 0.015"/>
       </geometry>
     </collision>
@@ -45,5 +45,5 @@
       <origin xyz="0 0 0.04" rpy="0 0 0"/>
       <geometry>
-        <box size="0.08 0.08 0.085"/>
+        <box size="0.09 0.09 0.09"/>
       </geometry>
     </collision>
@@ -76,5 +76,5 @@
       <origin xyz="0 0 0.175" rpy="0 0 0"/>
       <geometry>
-        <box size="0.06 0.06 0.35"/>
+        <box size="0.07 0.07 0.355"/>
       </geometry>
     </collision>
@@ -107,5 +107,5 @@
       <origin xyz="0.11 0 0" rpy="0 0 0"/>
       <geometry>
-        <box size="0.22 0.06 0.06"/>
+        <box size="0.23 0.07 0.07"/>
       </geometry>
     </collision>
@@ -138,5 +138,5 @@
       <origin xyz="0.03 0 0" rpy="0 0 0"/>
       <geometry>
-        <box size="0.06 0.04 0.04"/>
+        <box size="0.07 0.05 0.05"/>
       </geometry>
     </collision>
@@ -169,5 +169,5 @@
       <origin xyz="0.035 0 0" rpy="0 0 0"/>
       <geometry>
-        <box size="0.07 0.04 0.04"/>
+        <box size="0.08 0.05 0.05"/>
       </geometry>
     </collision>
@@ -200,5 +200,5 @@
       <origin xyz="0.048 0 0" rpy="0 0 0"/>
       <geometry>
-        <box size="0.097 0.04 0.04"/>
+        <box size="0.107 0.05 0.05"/>
       </geometry>
     </collision>
@@ -231,5 +231,5 @@
       <origin xyz="0.024 0 0" rpy="0 0 0"/>
       <geometry>
-        <box size="0.05 0.04 0.04"/>
+        <box size="0.06 0.05 0.05"/>
       </geometry>
     </collision>

File: src/chassis_description/urdf/chassis.xacro (robot description, xacro)
@@ -2,14 +2,21 @@
 <robot xmlns:xacro="http://www.ros.org/wiki/xacro">
   <!-- ==================== chassis_link (Main Body) ==================== -->
+  <link name="chassis_base_link" />
+  <joint name="chassis_base_to_chassis_joint" type="fixed">
+    <origin xyz="0 0 0.1" rpy="0 0 0"/>
+    <parent link="chassis_base_link"/>
+    <child link="chassis_link"/>
+  </joint>
+  <!-- ==================== chassis_link (Main Body) ==================== -->
   <link name="chassis_link">
     <inertial>
-      <origin xyz="0 0 0.1" rpy="0 0 0"/>
+      <origin xyz="0 0 0" rpy="0 0 0"/>
       <mass value="10.0"/>
       <inertia ixx="0.5" ixy="0" ixz="0" iyy="0.5" iyz="0" izz="0.5"/>
     </inertial>
     <visual>
-      <origin xyz="0 0 0.1" rpy="0 0 0"/>
+      <origin xyz="0 0 0" rpy="0 0 0"/>
       <geometry>
-        <box size="0.6 0.6 0.2"/>
+        <box size="0.6 0.6 0.1"/>
       </geometry>
       <material name="chassis_color">
@@ -18,7 +25,7 @@
     </visual>
     <collision>
-      <origin xyz="0 0 0.1" rpy="0 0 0"/>
+      <origin xyz="0 0 0" rpy="0 0 0"/>
       <geometry>
-        <box size="0.6 0.6 0.2"/>
+        <box size="0.6 0.6 0.1"/>
       </geometry>
     </collision>
@@ -27,13 +34,13 @@
   <link name="armor_left_link">
     <visual>
-      <geometry><box size="0.4 0.02 0.2"/></geometry>
-      <material name="armor_color"><color rgba="1 0 0 1"/></material>
+      <geometry><box size="0.135 0.1 0.2"/></geometry>
+      <material name="armor_color"><color rgba="0.5 0.5 0.5 1"/></material>
     </visual>
     <collision>
-      <geometry><box size="0.4 0.02 0.2"/></geometry>
+      <geometry><box size="0.135 0.1 0.2"/></geometry>
     </collision>
   </link>
   <joint name="joint_armor_left" type="fixed">
-    <origin xyz="0 0.21 0.1" rpy="0 0 0"/>
+    <origin xyz="0 -0.25 0.15" rpy="0 0 0"/>
     <parent link="chassis_link"/>
     <child link="armor_left_link"/>
@@ -42,13 +49,13 @@
   <link name="armor_right_link">
     <visual>
-      <geometry><box size="0.1 0.135 0.2"/></geometry>
+      <geometry><box size="0.135 0.1 0.2"/></geometry>
       <material name="armor_color"/>
     </visual>
     <collision>
-      <geometry><box size="0.1 0.135 0.2"/></geometry>
+      <geometry><box size="0.135 0.1 0.2"/></geometry>
     </collision>
   </link>
   <joint name="joint_armor_right" type="fixed">
-    <origin xyz="0 -0.21 0.1" rpy="0 0 0"/>
+    <origin xyz="0 0.25 0.15" rpy="0 0 0"/>
     <parent link="chassis_link"/>
     <child link="armor_right_link"/>
@@ -57,13 +64,13 @@
   <link name="warehouse_big_link">
     <visual>
-      <geometry><box size="0.19 0.46 0.25"/></geometry>
+      <geometry><box size="0.2 0.46 0.15"/></geometry>
       <material name="warehouse_color"><color rgba="0.4 0.4 0.4 1"/></material>
     </visual>
     <collision>
-      <geometry><box size="0.19 0.46 0.25"/></geometry>
+      <geometry><box size="0.2 0.46 0.15"/></geometry>
     </collision>
   </link>
   <joint name="joint_warehouse_big" type="fixed">
-    <origin xyz="-0.2 0 0.275" rpy="0 0 0"/>
+    <origin xyz="-0.2 0 0.125" rpy="0 0 0"/>
     <parent link="chassis_link"/>
     <child link="warehouse_big_link"/>
@@ -72,13 +79,13 @@
   <link name="warehouse_small_link">
     <visual>
-      <geometry><box size="0.13 0.19 0.14"/></geometry>
+      <geometry><box size="0.13 0.19 0.0933"/></geometry>
       <material name="warehouse_color"/>
     </visual>
     <collision>
-      <geometry><box size="0.13 0.19 0.14"/></geometry>
+      <geometry><box size="0.13 0.19 0.0933"/></geometry>
     </collision>
   </link>
   <joint name="joint_warehouse_small" type="fixed">
-    <origin xyz="-0.05 0 0.25" rpy="0 0 0"/>
+    <origin xyz="-0.05 0 0.09665" rpy="0 0 0"/>
     <parent link="chassis_link"/>
     <child link="warehouse_small_link"/>
@@ -94,11 +101,13 @@
     </visual>
     <collision>
-      <origin xyz="0.05 0 -0.05" rpy="0 0 0"/>
-      <geometry><box size="0.1 0.02 0.3"/></geometry>
+      <origin xyz="0 0 0" rpy="0 0 0"/>
+      <geometry>
+        <mesh filename="package://chassis_description/meshes/left.STL"/>
+      </geometry>
     </collision>
   </link>
   <joint name="joint_left_mesh" type="fixed">
-    <origin xyz="-0.34589 0.1785 0.17728" rpy="0 0 0"/>
-    <parent link="chassis_link"/>
+    <origin xyz="-0.05 -0.18 0.125" rpy="0 0 0"/>
+    <parent link="warehouse_big_link"/>
     <child link="left"/>
   </joint>
@@ -113,12 +122,29 @@
     </visual>
     <collision>
-      <origin xyz="0.05 0 -0.05" rpy="0 0 0"/>
-      <geometry><box size="0.1 0.02 0.3"/></geometry>
+      <origin xyz="0 0 0" rpy="0 0 0"/>
+      <geometry>
+        <mesh filename="package://chassis_description/meshes/right.STL"/>
+      </geometry>
     </collision>
   </link>
   <joint name="joint_right_mesh" type="fixed">
-    <origin xyz="-0.34589 -0.1785 0.17728" rpy="0 0 0"/>
-    <parent link="chassis_link"/>
+    <origin xyz="-0.05 0.18 0.125" rpy="0 0 0"/>
+    <parent link="warehouse_big_link"/>
     <child link="right"/>
   </joint>
+  <!-- ==================== 灯条 ==================== -->
+  <link name="light_link">
+    <visual>
+      <geometry><box size="0.06 0.285 0.07"/></geometry>
+      <material name="warehouse_color"><color rgba="0.4 0.4 0.4 1"/></material>
+    </visual>
+    <collision>
+      <geometry><box size="0.06 0.285 0.07"/></geometry>
+    </collision>
+  </link>
+  <joint name="joint_light" type="fixed">
+    <origin xyz="-0.07 0 0.11" rpy="0 0 0"/>
+    <parent link="warehouse_big_link"/>
+    <child link="light_link"/>
+  </joint>
 </robot>

File: src/gripper_description/urdf/gripper.xacro (robot description, xacro)
@@ -117,3 +117,10 @@
     <limit lower="0" upper="0.04" effort="2" velocity="2"/>
   </joint>
+  <!-- ==================== link_ee (End Effector) ==================== -->
+  <link name="link_ee"/>
+  <joint name="joint_ee" type="fixed">
+    <origin xyz="0.13 0 0" rpy="0 0 0"/>
+    <parent link="gripper_base_link"/>
+    <child link="link_ee"/>
+  </joint>
 </robot>

File: src/my_robot_description/urdf/my_robot.urdf.xacro (robot description, xacro)
@@ -9,5 +9,5 @@
   <!-- Connect chassis to arm -->
   <joint name="chassis_to_arm_joint" type="fixed">
-    <origin xyz="0.15 0 0.2" rpy="0 0 0"/>
+    <origin xyz="0.15 0 0.05" rpy="0 0 0"/>
     <parent link="chassis_link"/>
     <child link="base_link"/>

Commit message: 可以控制了

File: src/arm_description/urdf/arm.xacro (robot description, xacro)
@@ -85,5 +85,5 @@
     <child link="Link_2"/>
     <axis xyz="0 -1 0"/>
-    <limit lower="-0.2618" upper="1.1345" effort="20" velocity="2"/>
+    <limit lower="-0.262" upper="1.134" effort="20" velocity="2"/>
   </joint>
   <!-- ==================== Link3 ==================== -->

File: src/gripper_description/urdf/gripper.xacro (robot description, xacro)
@@ -124,3 +124,10 @@
     <child link="link_ee"/>
   </joint>
+  <!-- ==================== gripper_center (TCP) ==================== -->
+  <link name="gripper_center"/>
+  <joint name="joint_gripper_center" type="fixed">
+    <origin xyz="0.10 0 0" rpy="0 0 0"/>
+    <parent link="gripper_base_link"/>
+    <child link="gripper_center"/>
+  </joint>
 </robot>
