Commit message: 实现FDCC

File: src/arm_description/urdf/arm.ros2_control.xacro (robot description, xacro)
@@ -1,5 +1,5 @@
 <?xml version="1.0"?>
 <robot xmlns:xacro="http://www.ros.org/wiki/xacro">
-  <xacro:macro name="arm_ros2_control" params="name use_mock_hardware:=false gravity_compensation_mode:=off active_real_joints:='' can0_interface:=can0 can1_interface:=can1">
+  <xacro:macro name="arm_ros2_control" params="name use_mock_hardware:=false gravity_compensation_mode:=off active_real_joints:='' can0_interface:=can0 can1_interface:=can1 robot_description_file:=/tmp/robot_description.urdf">
     <ros2_control name="${name}" type="system">
       <hardware>
@@ -10,5 +10,5 @@
           <plugin>arm_hardware_interface/ArmHardwareInterface</plugin>
         </xacro:unless>
-        <param name="robot_description">$(find my_robot_description)/urdf/my_robot.urdf.xacro</param>
+        <param name="robot_description">${robot_description_file}</param>
         <param name="gravity_compensation_mode">${gravity_compensation_mode}</param>
         <param name="active_real_joints">${active_real_joints}</param>

File: src/my_robot_description/urdf/my_robot.urdf.xacro (robot description, xacro)
@@ -12,4 +12,5 @@
   <xacro:arg name="can0_interface" default="can0"/>
   <xacro:arg name="can1_interface" default="can1"/>
+  <xacro:arg name="robot_description_file" default="/tmp/robot_description.urdf"/>
   <!-- Include ros2_control configuration -->
   <xacro:include filename="$(find arm_description)/urdf/arm.ros2_control.xacro"/>
@@ -19,5 +20,6 @@
     gravity_compensation_mode="$(arg gravity_compensation_mode)"
     can0_interface="$(arg can0_interface)"
-    can1_interface="$(arg can1_interface)"/>
+    can1_interface="$(arg can1_interface)"
+    robot_description_file="$(arg robot_description_file)"/>
   <!-- Connect chassis to arm -->
   <joint name="chassis_to_arm_joint" type="fixed">

Commit message: ``` docs: 删除过时的文档文件并更新URDF支持多版本
删除了以下过时的文档文件：
- MIGRATE_MINIPC.md
- README.md
- README_real_robot.md
- SESSION_CHANGES_20260701.md

同时更新了URDF文件以支持多版本机械臂：
- 修改arm.xacro支持arm_version参数
- 将原有的arm_links.xacro和arm_joints.xacro拆分为V1.0和V1.1版本
- 更新arm.ros2_control.xacro支持接收arm_version参数并动态调整关节限位
- 为damiao_motor添加recv_can_id配置以支持更灵活的CAN反馈匹配
```

File: src/arm_description/urdf/arm.ros2_control.xacro (robot description, xacro)
@@ -1,5 +1,6 @@
 <?xml version="1.0"?>
 <robot xmlns:xacro="http://www.ros.org/wiki/xacro">
-  <xacro:macro name="arm_ros2_control" params="name use_mock_hardware:=false gravity_compensation_mode:=off active_real_joints:='' can0_interface:=can0 can1_interface:=can1 robot_description_file:=/tmp/robot_description.urdf">
+  <xacro:macro name="arm_ros2_control" params="name arm_version:=v1_0 use_mock_hardware:=false gravity_compensation_mode:=off active_real_joints:='' can0_interface:=can0 can1_interface:=can1 robot_description_file:=/tmp/robot_description.urdf">
+    <xacro:property name="is_arm_v1_1" value="${arm_version == 'v1_1' or arm_version == 'v1.1' or arm_version == '1.1' or arm_version == 1.1}"/>
     <ros2_control name="${name}" type="system">
       <hardware>
@@ -24,4 +25,5 @@
         <state_interface name="effort"/>
         <param name="can_id">1</param>
+        <param name="recv_can_id">0x11</param>
         <param name="motor_model">J8009</param>
         <param name="can_bus">${can0_interface}</param>
@@ -44,6 +46,6 @@
         <param name="kp">120.0</param>
         <param name="kd">3.0</param>
-        <param name="lower_limit">-0.262</param>
-        <param name="upper_limit">1.134</param>
+        <param name="lower_limit">${-1.204 if is_arm_v1_1 else -0.262}</param>
+        <param name="upper_limit">${0.262 if is_arm_v1_1 else 1.134}</param>
       </joint>
       <joint name="joint3">
@@ -60,5 +62,5 @@
         <param name="kd">3.0</param>
         <param name="lower_limit">-0.9599</param>
-        <param name="upper_limit">0.9599</param>
+        <param name="upper_limit">${1.221 if is_arm_v1_1 else 0.9599}</param>
       </joint>
       <joint name="joint4">
@@ -90,5 +92,5 @@
         <param name="kp">120.0</param>
         <param name="kd">3.0</param>
-        <param name="lower_limit">-1.5708</param>
+        <param name="lower_limit">${-0.78 if is_arm_v1_1 else -1.5708}</param>
         <param name="upper_limit">1.5708</param>
         <param name="direction">-1.0</param>

File: src/arm_description/urdf/arm.xacro (robot description, xacro)
@@ -3,14 +3,24 @@
   Arm Description — 7-DOF 机械臂 URDF 入口文件
   子文件结构（对标 OpenArm 的模块化组织）：
-    arm_links.xacro   — 全部 link 定义（惯量、视觉、碰撞）
-    arm_joints.xacro  — 全部 joint 定义（限位、运动学）
+    variants/V1.0/arm_links_v1_0.xacro   — v1.0 link 定义（惯量、视觉、碰撞）
+    variants/V1.0/arm_joints_v1_0.xacro  — v1.0 joint 定义（限位、运动学）
+    variants/V1.1/arm_links_v1_1.xacro   — v1.1 link 定义
+    variants/V1.1/arm_joints_v1_1.xacro  — v1.1 joint 定义
     arm.ros2_control.xacro  — ros2_control 硬件接口与控制器参数
   用法：
-    xacro arm.xacro
+    xacro arm.xacro arm_version:=v1_0
+    xacro arm.xacro arm_version:=v1_1
 -->
 <robot name="arm" xmlns:xacro="http://www.ros.org/wiki/xacro">
-  <!-- Links -->
-  <xacro:include filename="$(find arm_description)/urdf/arm_links.xacro"/>
-  <!-- Joints -->
-  <xacro:include filename="$(find arm_description)/urdf/arm_joints.xacro"/>
+  <xacro:arg name="arm_version" default="v1_0"/>
+  <!-- v1.0: current production geometry/dynamics. Accept "1.0" as an alias. -->
+  <xacro:if value="$(eval arm_version == 'v1_0' or arm_version == 'v1.0' or arm_version == '1.0' or arm_version == 1.0)">
+    <xacro:include filename="$(find arm_description)/urdf/variants/V1.0/arm_links_v1_0.xacro"/>
+    <xacro:include filename="$(find arm_description)/urdf/variants/V1.0/arm_joints_v1_0.xacro"/>
+  </xacro:if>
+  <!-- v1.1: prepared variant. Files currently mirror v1.0 until the new J5-J7 model is added. -->
+  <xacro:if value="$(eval arm_version == 'v1_1' or arm_version == 'v1.1' or arm_version == '1.1' or arm_version == 1.1)">
+    <xacro:include filename="$(find arm_description)/urdf/variants/V1.1/arm_links_v1_1.xacro"/>
+    <xacro:include filename="$(find arm_description)/urdf/variants/V1.1/arm_joints_v1_1.xacro"/>
+  </xacro:if>
 </robot>

File: src/chassis_description/urdf/chassis.xacro (robot description, xacro)
@@ -1,150 +1,15 @@
 <?xml version="1.0"?>
+<!--
+  Chassis Description entrypoint.
+  v1_0 is the current production chassis. v1_1 is prepared as a separate
+  variant so the new chassis can be integrated without changing launch files.
+-->
 <robot xmlns:xacro="http://www.ros.org/wiki/xacro">
-  <!-- ==================== chassis_link (Main Body) ==================== -->
-  <link name="chassis_base_link" />
-  <joint name="chassis_base_to_chassis_joint" type="fixed">
-    <origin xyz="0 0 0.1" rpy="0 0 0"/>
-    <parent link="chassis_base_link"/>
-    <child link="chassis_link"/>
-  </joint>
-  <!-- ==================== chassis_link (Main Body) ==================== -->
-  <link name="chassis_link">
-    <inertial>
-      <origin xyz="0 0 0" rpy="0 0 0"/>
-      <mass value="10.0"/>
-      <inertia ixx="0.5" ixy="0" ixz="0" iyy="0.5" iyz="0" izz="0.5"/>
-    </inertial>
-    <visual>
-      <origin xyz="0 0 0" rpy="0 0 0"/>
-      <geometry>
-        <box size="0.6 0.6 0.1"/>
-      </geometry>
-      <material name="chassis_color">
-        <color rgba="0.2 0.2 0.2 1"/>
-      </material>
-    </visual>
-    <collision>
-      <origin xyz="0 0 0" rpy="0 0 0"/>
-      <geometry>
-        <box size="0.6 0.6 0.1"/>
-      </geometry>
-    </collision>
-  </link>
-  <!-- ==================== armor_left_link ==================== -->
-  <link name="armor_left_link">
-    <visual>
-      <geometry><box size="0.135 0.1 0.2"/></geometry>
-      <material name="armor_color"><color rgba="0.5 0.5 0.5 1"/></material>
-    </visual>
-    <collision>
-      <geometry><box size="0.135 0.1 0.2"/></geometry>
-    </collision>
-  </link>
-  <joint name="joint_armor_left" type="fixed">
-    <origin xyz="0 -0.25 0.15" rpy="0 0 0"/>
-    <parent link="chassis_link"/>
-    <child link="armor_left_link"/>
-  </joint>
-  <!-- ==================== armor_right_link ==================== -->
-  <link name="armor_right_link">
-    <visual>
-      <geometry><box size="0.135 0.1 0.2"/></geometry>
-      <material name="armor_color"/>
-    </visual>
-    <collision>
-      <geometry><box size="0.135 0.1 0.2"/></geometry>
-    </collision>
-  </link>
-  <joint name="joint_armor_right" type="fixed">
-    <origin xyz="0 0.25 0.15" rpy="0 0 0"/>
-    <parent link="chassis_link"/>
-    <child link="armor_right_link"/>
-  </joint>
-  <!-- ==================== warehouse_big_link ==================== -->
-  <link name="warehouse_big_link">
-    <visual>
-      <geometry><box size="0.2 0.46 0.15"/></geometry>
-      <material name="warehouse_color"><color rgba="0.4 0.4 0.4 1"/></material>
-    </visual>
-    <collision>
-      <geometry><box size="0.2 0.46 0.15"/></geometry>
-    </collision>
-  </link>
-  <joint name="joint_warehouse_big" type="fixed">
-    <origin xyz="-0.2 0 0.125" rpy="0 0 0"/>
-    <parent link="chassis_link"/>
-    <child link="warehouse_big_link"/>
-  </joint>
-  <!-- ==================== warehouse_small_link ==================== -->
-  <link name="warehouse_small_link">
-    <visual>
-      <geometry><box size="0.13 0.19 0.0933"/></geometry>
-      <material name="warehouse_color"/>
-    </visual>
-    <collision>
-      <geometry><box size="0.13 0.19 0.0933"/></geometry>
-    </collision>
-  </link>
-  <joint name="joint_warehouse_small" type="fixed">
-    <origin xyz="-0.05 0 0.09665" rpy="0 0 0"/>
-    <parent link="chassis_link"/>
-    <child link="warehouse_small_link"/>
-  </joint>
-  <!-- ==================== left link (Original Mesh) ==================== -->
-  <link name="left">
-    <visual>
-      <origin xyz="0 0 0" rpy="0 0 0"/>
-      <geometry>
-        <mesh filename="package://chassis_description/meshes/left.STL"/>
-      </geometry>
-      <material name="cyan"><color rgba="0 1 1 1"/></material>
-    </visual>
-    <collision>
-      <origin xyz="0 0 0" rpy="0 0 0"/>
-      <geometry>
-        <mesh filename="package://chassis_description/meshes/left.STL"/>
-      </geometry>
-    </collision>
-  </link>
-  <joint name="joint_left_mesh" type="fixed">
-    <origin xyz="-0.05 -0.18 0.125" rpy="0 0 0"/>
-    <parent link="warehouse_big_link"/>
-    <child link="left"/>
-  </joint>
-  <!-- ==================== right link (Original Mesh) ==================== -->
-  <link name="right">
-    <visual>
-      <origin xyz="0 0 0" rpy="0 0 0"/>
-      <geometry>
-        <mesh filename="package://chassis_description/meshes/right.STL"/>
-      </geometry>
-      <material name="white"><color rgba="1 1 1 1"/></material>
-    </visual>
-    <collision>
-      <origin xyz="0 0 0" rpy="0 0 0"/>
-      <geometry>
-        <mesh filename="package://chassis_description/meshes/right.STL"/>
-      </geometry>
-    </collision>
-  </link>
-  <joint name="joint_right_mesh" type="fixed">
-    <origin xyz="-0.05 0.18 0.125" rpy="0 0 0"/>
-    <parent link="warehouse_big_link"/>
-    <child link="right"/>
-  </joint>
-  <!-- ==================== 灯条 ==================== -->
-  <link name="light_link">
-    <visual>
-      <geometry><box size="0.06 0.285 0.07"/></geometry>
-      <material name="warehouse_color"><color rgba="0.4 0.4 0.4 1"/></material>
-    </visual>
-    <collision>
-      <geometry><box size="0.06 0.285 0.07"/></geometry>
-    </collision>
-  </link>
-  <joint name="joint_light" type="fixed">
-    <origin xyz="-0.07 0 0.11" rpy="0 0 0"/>
-    <parent link="warehouse_big_link"/>
-    <child link="light_link"/>
-  </joint>
+  <xacro:arg name="chassis_version" default="v1_0"/>
+  <xacro:if value="$(eval chassis_version == 'v1_0' or chassis_version == 'v1.0' or chassis_version == '1.0' or chassis_version == 1.0)">
+    <xacro:include filename="$(find chassis_description)/urdf/variants/V1.0/chassis_v1_0.xacro"/>
+  </xacro:if>
+  <xacro:if value="$(eval chassis_version == 'v1_1' or chassis_version == 'v1.1' or chassis_version == '1.1' or chassis_version == 1.1)">
+    <xacro:include filename="$(find chassis_description)/urdf/variants/V1.1/chassis_v1_1.xacro"/>
+  </xacro:if>
 </robot>

File: src/gripper_description/urdf/gripper.xacro (robot description, xacro)
@@ -1,133 +1,11 @@
 <?xml version="1.0"?>
+<!-- Gripper Description entrypoint. -->
 <robot xmlns:xacro="http://www.ros.org/wiki/xacro">
-  <!-- ==================== gripper_base_link ==================== -->
-  <link name="gripper_base_link">
-    <inertial>
-      <origin xyz="0.024119 -0.00025348 1.4037E-05" rpy="0 0 0"/>
-      <mass value="0.10268"/>
-      <inertia ixx="4.2026E-05" ixy="-4.1834E-08" ixz="-5.3192E-10"
-               iyy="3.0131E-05" iyz="2.7197E-08" izz="3.0109E-05"/>
-    </inertial>
-    <visual>
-      <origin xyz="0 0 0" rpy="0 0 0"/>
-      <geometry>
-        <mesh filename="package://gripper_description/meshes/gripper_base_link.STL"/>
-      </geometry>
-      <material name="">
-        <color rgba="0.79216 0.81961 0.93333 1"/>
-      </material>
-    </visual>
-    <collision>
-      <origin xyz="0 0 0" rpy="0 0 0"/>
-      <geometry>
-        <mesh filename="package://gripper_description/meshes/gripper_base_link.STL"/>
-      </geometry>
-    </collision>
-  </link>
-  <!-- ==================== grippeer_Link (gripper body) ==================== -->
-  <link name="grippeer_Link">
-    <inertial>
-      <origin xyz="0.040428 -0.00017354 1.2493E-05" rpy="0 0 0"/>
-      <mass value="0.093865"/>
-      <inertia ixx="0.00022061" ixy="1.0893E-19" ixz="3.8261E-21"
-               iyy="2.9769E-05" iyz="-2.4504E-16" izz="0.00019995"/>
-    </inertial>
-    <visual>
-      <origin xyz="0 0 0" rpy="0 0 0"/>
-      <geometry>
-        <mesh filename="package://gripper_description/meshes/grippeer_Link.STL"/>
-      </geometry>
-      <material name="">
-        <color rgba="0.79216 0.81961 0.93333 1"/>
-      </material>
-    </visual>
-    <collision>
-      <origin xyz="0 0 0" rpy="0 0 0"/>
-      <geometry>
-        <mesh filename="package://gripper_description/meshes/grippeer_Link.STL"/>
-      </geometry>
-    </collision>
-  </link>
-  <joint name="joint_gripper" type="fixed">
-    <origin xyz="0 0 0" rpy="0 0 0"/>
-    <parent link="gripper_base_link"/>
-    <child link="grippeer_Link"/>
-  </joint>
-  <!-- ==================== right_finger_Link ==================== -->
-  <link name="right_finger_Link">
-    <inertial>
-      <origin xyz="0.032482 0.0068743 0.00084038" rpy="0 0 0"/>
-      <mass value="0.095586"/>
-      <inertia ixx="2.0674E-05" ixy="-5.6199E-06" ixz="-1.1351E-08"
-               iyy="9.0681E-05" iyz="4.7589E-08" izz="0.0001011"/>
-    </inertial>
-    <visual>
-      <origin xyz="0 0 0" rpy="0 0 0"/>
-      <geometry>
-        <mesh filename="package://gripper_description/meshes/right_finger_Link.STL"/>
-      </geometry>
-      <material name="">
-        <color rgba="0.79216 0.81961 0.93333 1"/>
-      </material>
-    </visual>
-    <collision>
-      <origin xyz="0 0 0" rpy="0 0 0"/>
-      <geometry>
-        <mesh filename="package://gripper_description/meshes/right_finger_Link.STL"/>
-      </geometry>
-    </collision>
-  </link>
-  <joint name="joint_right_finger" type="prismatic">
-    <origin xyz="0.071 0.059926 1.2493E-05" rpy="0 0 0"/>
-    <parent link="grippeer_Link"/>
-    <child link="right_finger_Link"/>
-    <axis xyz="0 1 0"/>
-    <limit lower="-0.04" upper="0" effort="2" velocity="2"/>
-  </joint>
-  <!-- ==================== left_finger_Link ==================== -->
-  <link name="left_finger_Link">
-    <inertial>
-      <origin xyz="0.032717 -0.0068743 -0.00084038" rpy="0 0 0"/>
-      <mass value="0.095586"/>
-      <inertia ixx="2.0674E-05" ixy="5.6199E-06" ixz="1.1351E-08"
-               iyy="9.0681E-05" iyz="4.7589E-08" izz="0.0001011"/>
-    </inertial>
-    <visual>
-      <origin xyz="0 0 0" rpy="0 0 0"/>
-      <geometry>
-        <mesh filename="package://gripper_description/meshes/left_finger_Link.STL"/>
-      </geometry>
-      <material name="">
-        <color rgba="0.79216 0.81961 0.93333 1"/>
-      </material>
-    </visual>
-    <collision>
-      <origin xyz="0 0 0" rpy="0 0 0"/>
-      <geometry>
-        <mesh filename="package://gripper_description/meshes/left_finger_Link.STL"/>
-      </geometry>
-    </collision>
-  </link>
-  <joint name="joint_left_finger" type="prismatic">
-    <origin xyz="0.071 -0.060274 1.2493E-05" rpy="0 0 0"/>
-    <parent link="grippeer_Link"/>
-    <child link="left_finger_Link"/>
-    <axis xyz="0 1 0"/>
-    <mimic joint="joint_right_finger" multiplier="-1.0" offset="0"/>
-    <limit lower="0" upper="0.04" effort="2" velocity="2"/>
-  </joint>
-  <!-- ==================== link_ee (End Effector) ==================== -->
-  <link name="link_ee"/>
-  <joint name="joint_ee" type="fixed">
-    <origin xyz="0.13 0 0" rpy="0 0 0"/>
-    <parent link="gripper_base_link"/>
-    <child link="link_ee"/>
-  </joint>
-  <!-- ==================== gripper_center (TCP) ==================== -->
-  <link name="gripper_center"/>
-  <joint name="joint_gripper_center" type="fixed">
-    <origin xyz="0.10 0 0" rpy="0 0 0"/>
-    <parent link="gripper_base_link"/>
-    <child link="gripper_center"/>
-  </joint>
+  <xacro:arg name="gripper_version" default="v1_0"/>
+  <xacro:if value="$(eval gripper_version == 'v1_0' or gripper_version == 'v1.0' or gripper_version == '1.0' or gripper_version == 1.0)">
+    <xacro:include filename="$(find gripper_description)/urdf/variants/V1.0/gripper_v1_0.xacro"/>
+  </xacro:if>
+  <xacro:if value="$(eval gripper_version == 'v1_1' or gripper_version == 'v1.1' or gripper_version == '1.1' or gripper_version == 1.1)">
+    <xacro:include filename="$(find gripper_description)/urdf/variants/V1.1/gripper_v1_1.xacro"/>
+  </xacro:if>
 </robot>

File: src/my_robot_description/urdf/my_robot.urdf.xacro (robot description, xacro)
@@ -1,11 +1,8 @@
 <?xml version="1.0"?>
 <robot name="my_robot" xmlns:xacro="http://www.ros.org/wiki/xacro">
-  <!-- Include arm description -->
-  <xacro:include filename="$(find arm_description)/urdf/arm.xacro"/>
-  <!-- Include gripper description -->
-  <xacro:include filename="$(find gripper_description)/urdf/gripper.xacro"/>
-  <!-- Include chassis description -->
-  <xacro:include filename="$(find chassis_description)/urdf/chassis.xacro"/>
   <!-- Arguments -->
+  <xacro:arg name="arm_version" default="v1_0"/>
+  <xacro:arg name="chassis_version" default="v1_0"/>
+  <xacro:arg name="gripper_version" default="v1_0"/>
   <xacro:arg name="use_mock_hardware" default="false"/>
   <xacro:arg name="gravity_compensation_mode" default="off"/>
@@ -13,8 +10,15 @@
   <xacro:arg name="can1_interface" default="can1"/>
   <xacro:arg name="robot_description_file" default="/tmp/robot_description.urdf"/>
+  <!-- Include gripper description -->
+  <xacro:include filename="$(find gripper_description)/urdf/gripper.xacro"/>
+  <!-- Include chassis description -->
+  <xacro:include filename="$(find chassis_description)/urdf/chassis.xacro"/>
+  <!-- Include arm description after arm_version is declared. -->
+  <xacro:include filename="$(find arm_description)/urdf/arm.xacro"/>
   <!-- Include ros2_control configuration -->
   <xacro:include filename="$(find arm_description)/urdf/arm.ros2_control.xacro"/>
   <xacro:arm_ros2_control
     name="ArmControl"
+    arm_version="$(arg arm_version)"
     use_mock_hardware="$(arg use_mock_hardware)"
     gravity_compensation_mode="$(arg gravity_compensation_mode)"
@@ -28,10 +32,20 @@
     <child link="base_link"/>
   </joint>
-  <!-- Connect gripper to arm: gripper_base_link attached to tool_link -->
-  <joint name="gripper_base_joint" type="fixed">
-    <parent link="tool_link"/>
-    <child link="gripper_base_link"/>
-    <origin xyz="0 0 0" rpy="0 0 0"/>
-  </joint>
+  <!-- V1.0 gripper is attached to the arm-provided tool_link. -->
+  <xacro:if value="$(eval gripper_version == 'v1_0' or gripper_version == 'v1.0' or gripper_version == '1.0' or gripper_version == 1.0)">
+    <joint name="gripper_base_joint" type="fixed">
+      <parent link="tool_link"/>
+      <child link="gripper_base_link"/>
+      <origin xyz="0 0 0" rpy="0 0 0"/>
+    </joint>
+  </xacro:if>
+  <!-- V1.1 gripper owns the end effector and tool frame. -->
+  <xacro:if value="$(eval gripper_version == 'v1_1' or gripper_version == 'v1.1' or gripper_version == '1.1' or gripper_version == 1.1)">
+    <joint name="gripper_base_joint" type="fixed">
+      <parent link="Link7"/>
+      <child link="gripper_base_link"/>
+      <origin xyz="0.056450 0 0" rpy="0 0 0"/>
+    </joint>
+  </xacro:if>
   <!-- Future: include chassis_description connection here -->
 </robot>

Commit message: fix(robot): 修复V1.1机械臂配置文件中的错误
修复了V1.1版本机械臂的关节限制参数错误，包括上下限值和旋转轴方向，
同时修正了启动脚本中错误的launch文件路径，并更新了相关配置文件的参数设置。

BREAKING CHANGE: 关节限制参数已更改，可能影响现有运动规划行为。

File: src/arm_description/urdf/arm.ros2_control.xacro (robot description, xacro)
@@ -46,6 +46,6 @@
         <param name="kp">120.0</param>
         <param name="kd">3.0</param>
-        <param name="lower_limit">${-1.204 if is_arm_v1_1 else -0.262}</param>
-        <param name="upper_limit">${0.262 if is_arm_v1_1 else 1.134}</param>
+        <param name="lower_limit">${-0.262 if is_arm_v1_1 else -0.262}</param>
+        <param name="upper_limit">${1.204 if is_arm_v1_1 else 1.134}</param>
       </joint>
       <joint name="joint3">

File: src/arm_description/urdf/variants/V1.1/arm_joints_v1_1.xacro (robot description, xacro)
@@ -15,6 +15,6 @@
     <parent link="Link_1" />
     <child link="Link_2" />
-    <axis xyz="0 1 0" />
-    <limit lower="-1.204" upper="0.262" effort="20" velocity="2" />
+    <axis xyz="0 -1 0" />
+    <limit lower="-0.262" upper="1.204" effort="20" velocity="2" />
   </joint>
   <!-- ==================== J3: Link_2 → Link_3 ==================== -->
