Commit message: feat(arm_hardware): 添加重力补偿功能和调试接口
- 添加 gravity_compensation_mode 和 gravity_effort_scale 参数支持
- 实现重力补偿器初始化和模式切换功能
- 新增多个调试话题用于监控原始电机状态、处理后的关节状态和重力补偿力矩
- 添加 DLS 控制器和关节控制器的诊断功能

feat(can_motor): 扩展电机控制接口支持动态 Kp/Kd 配置

- 在 DMDeviceCollection 中新增 sendCommandsWithGains 方法
- 允许按电机单独设置 Kp/Kd 增益参数
- 更新电机状态结构体添加反馈计数统计

refactor(hardware_interface): 重构实时硬件接口的使能逻辑

- 实现 clear_errors_enable_and_wait 方法进行错误清除和电机使能
- 添加 all_real_motors_feedback_ok 方法检查电机反馈状态
- 优化电机同步控制流程

docs(can): 更新启动命令文档

File: src/arm_description/urdf/arm.ros2_control.xacro (robot description, xacro)
@@ -1,5 +1,5 @@
 <?xml version="1.0"?>
 <robot xmlns:xacro="http://www.ros.org/wiki/xacro">
-  <xacro:macro name="arm_ros2_control" params="name arm_version:=v1_0 use_mock_hardware:=false gravity_compensation_mode:=off active_real_joints:='' can0_interface:=can0 can1_interface:=can1 robot_description_file:=/tmp/robot_description.urdf">
+  <xacro:macro name="arm_ros2_control" params="name arm_version:=v1_0 use_mock_hardware:=false gravity_compensation_mode:=off gravity_effort_scale:=0.0 active_real_joints:='' can0_interface:=can0 can1_interface:=can1 robot_description_file:=/tmp/robot_description.urdf">
     <xacro:property name="is_arm_v1_1" value="${arm_version == 'v1_1' or arm_version == 'v1.1' or arm_version == '1.1' or arm_version == 1.1}"/>
     <ros2_control name="${name}" type="system">
@@ -13,4 +13,5 @@
         <param name="robot_description">${robot_description_file}</param>
         <param name="gravity_compensation_mode">${gravity_compensation_mode}</param>
+        <param name="gravity_effort_scale">${gravity_effort_scale}</param>
         <param name="active_real_joints">${active_real_joints}</param>
         <param name="j2j3_coupling">0.986</param>
@@ -44,5 +45,5 @@
         <param name="motor_model">J8009</param>
         <param name="can_bus">${can0_interface}</param>
-        <param name="kp">120.0</param>
+        <param name="kp">240.0</param>
         <param name="kd">3.0</param>
         <param name="lower_limit">${-0.262 if is_arm_v1_1 else -0.262}</param>
@@ -59,5 +60,5 @@
         <param name="motor_model">J8009</param>
         <param name="can_bus">${can0_interface}</param>
-        <param name="kp">120.0</param>
+        <param name="kp">240.0</param>
         <param name="kd">3.0</param>
         <param name="lower_limit">-0.9599</param>

File: src/my_robot_description/urdf/my_robot.urdf.xacro (robot description, xacro)
@@ -7,4 +7,6 @@
   <xacro:arg name="use_mock_hardware" default="false"/>
   <xacro:arg name="gravity_compensation_mode" default="off"/>
+  <xacro:arg name="gravity_effort_scale" default="0.0"/>
+  <xacro:arg name="active_real_joints" default=""/>
   <xacro:arg name="can0_interface" default="can0"/>
   <xacro:arg name="can1_interface" default="can1"/>
@@ -23,4 +25,6 @@
     use_mock_hardware="$(arg use_mock_hardware)"
     gravity_compensation_mode="$(arg gravity_compensation_mode)"
+    gravity_effort_scale="$(arg gravity_effort_scale)"
+    active_real_joints="$(arg active_real_joints)"
     can0_interface="$(arg can0_interface)"
     can1_interface="$(arg can1_interface)"

Commit message: 0726

File: src/arm_description/urdf/arm.ros2_control.xacro (robot description, xacro)
@@ -1,5 +1,5 @@
 <?xml version="1.0"?>
 <robot xmlns:xacro="http://www.ros.org/wiki/xacro">
-  <xacro:macro name="arm_ros2_control" params="name arm_version:=v1_0 use_mock_hardware:=false gravity_compensation_mode:=off gravity_effort_scale:=0.0 active_real_joints:='' can0_interface:=can0 can1_interface:=can1 robot_description_file:=/tmp/robot_description.urdf">
+  <xacro:macro name="arm_ros2_control" params="name arm_version:=v1_0 use_mock_hardware:=false gravity_compensation_mode:=off gravity_effort_scale:=0.0 j2j3_j3_gravity_effort_scale:=1.0 active_real_joints:='' can0_interface:=can0 can1_interface:=can1 robot_description_file:=/tmp/robot_description.urdf">
     <xacro:property name="is_arm_v1_1" value="${arm_version == 'v1_1' or arm_version == 'v1.1' or arm_version == '1.1' or arm_version == 1.1}"/>
     <ros2_control name="${name}" type="system">
@@ -16,4 +16,12 @@
         <param name="active_real_joints">${active_real_joints}</param>
         <param name="j2j3_coupling">0.986</param>
+        <param name="j2j3_j3_scale">1.0</param>
+        <param name="j2j3_j3_offset">0.0</param>
+        <param name="j2j3_poly_a3">0.0</param>
+        <param name="j2j3_poly_a2">0.0</param>
+        <param name="j2j3_poly_a1">0.0</param>
+        <param name="j2j3_poly_a0">0.0</param>
+        <param name="j2j3_scale_mode">divide</param>
+        <param name="j2j3_j3_gravity_effort_scale">${j2j3_j3_gravity_effort_scale}</param>
       </hardware>
       <!-- J1-J4 使用 CAN 总线 can0 -->
@@ -77,6 +85,6 @@
         <param name="kp">120.0</param>
         <param name="kd">3.0</param>
-        <param name="lower_limit">-2.3562</param>
-        <param name="upper_limit">2.3562</param>
+        <param name="lower_limit">${-3.1416 if is_arm_v1_1 else -2.3562}</param>
+        <param name="upper_limit">${3.1416 if is_arm_v1_1 else 2.3562}</param>
       </joint>
       <!-- J5-J7 使用 CAN 总线 can1 -->
@@ -124,8 +132,8 @@
         <param name="kp">60.0</param>
         <param name="kd">1.0</param>
-        <param name="lower_limit">-1.5708</param>
-        <param name="upper_limit">1.5708</param>
+        <param name="lower_limit">${-3.1416 if is_arm_v1_1 else -1.5708}</param>
+        <param name="upper_limit">${3.1416 if is_arm_v1_1 else 1.5708}</param>
       </joint>
-      <!-- 夹爪关节：一直包含，无 can_id 则由硬件接口自动按 Mock 处理 -->
+      <!-- 夹爪关节：4310 电机，挂在 can1，CAN ID/反馈 ID 均为 8 -->
       <joint name="joint_right_finger">
         <command_interface name="position"/>
@@ -133,6 +141,13 @@
         <state_interface name="position"/>
         <state_interface name="velocity"/>
+        <state_interface name="effort"/>
+        <param name="can_id">8</param>
+        <param name="recv_can_id">8</param>
+        <param name="motor_model">J4310</param>
+        <param name="can_bus">${can1_interface}</param>
+        <param name="kp">60.0</param>
+        <param name="kd">1.0</param>
         <param name="lower_limit">0.0</param>
-        <param name="upper_limit">0.04</param>
+        <param name="upper_limit">1.2</param>
       </joint>
     </ros2_control>

File: src/arm_description/urdf/variants/V1.1/arm_joints_v1_1.xacro (robot description, xacro)
@@ -32,5 +32,5 @@
     <child link="Link4" />
     <axis xyz="1 0 0" />
-    <limit lower="-2.3562" upper="2.3562" effort="9" velocity="2" />
+    <limit lower="-3.1416" upper="3.1416" effort="9" velocity="2" />
   </joint>
   <!-- ==================== J5: Link_4 → Link_5 ==================== -->
@@ -56,5 +56,5 @@
     <child link="Link7" />
     <axis xyz="1 0 0" />
-    <limit lower="-1.57" upper="1.57" effort="10" velocity="5" />
+    <limit lower="-3.1416" upper="3.1416" effort="10" velocity="5" />
   </joint>
 </robot>

File: src/arm_description/urdf/variants/V1.1/arm_links_v1_1.xacro (robot description, xacro)
@@ -2,4 +2,5 @@
 <robot xmlns:xacro="http://www.ros.org/wiki/xacro">
   <!--Arm v1.1 link definitions generated from src/V1.1urdf/robot.urdf.-->
+  <xacro:property name="v1_1_collision_scale" value="0.85" />
   <!-- ==================== base_link ==================== -->
   <link name="base_link" />
@@ -104,5 +105,5 @@
       <origin xyz="0.010497 0 0.104100" rpy="0 0 0" />
       <geometry>
-        <box size="0.104994 0.195400 0.125200" />
+        <box size="${0.104994 * v1_1_collision_scale} ${0.195400 * v1_1_collision_scale} ${0.125200 * v1_1_collision_scale}" />
       </geometry>
     </collision>
@@ -208,5 +209,5 @@
       <origin xyz="0 0.036500 0.174789" rpy="0 0 0" />
       <geometry>
-        <box size="0.094000 0.095000 0.439578" />
+        <box size="${0.094000 * v1_1_collision_scale} ${0.095000 * v1_1_collision_scale} ${0.439578 * v1_1_collision_scale}" />
       </geometry>
     </collision>
@@ -357,5 +358,5 @@
       <origin xyz="0.109111 -0.037850 0.001500" rpy="0 0 0" />
       <geometry>
-        <box size="0.281777 0.108000 0.083000" />
+        <box size="${0.281777 * v1_1_collision_scale} ${0.108000 * v1_1_collision_scale} ${0.083000 * v1_1_collision_scale}" />
       </geometry>
     </collision>
@@ -434,5 +435,5 @@
       <origin xyz="0.055625 -0.001600 0" rpy="0 0 0" />
       <geometry>
-        <box size="0.055750 0.063200 0.070000" />
+        <box size="${0.055750 * v1_1_collision_scale} ${0.063200 * v1_1_collision_scale} ${0.070000 * v1_1_collision_scale}" />
       </geometry>
     </collision>
@@ -484,5 +485,5 @@
       <origin xyz="0.066883 0.038200 0.080585" rpy="0 0 0" />
       <geometry>
-        <box size="0.065093 0.066000 0.063730" />
+        <box size="${0.065093 * v1_1_collision_scale} ${0.066000 * v1_1_collision_scale} ${0.063730 * v1_1_collision_scale}" />
       </geometry>
     </collision>
@@ -534,5 +535,5 @@
       <origin xyz="0.036500 0 -0.035500" rpy="0 0 0" />
       <geometry>
-        <box size="0.028000 0.051999 0.082000" />
+        <box size="${0.028000 * v1_1_collision_scale} ${0.051999 * v1_1_collision_scale} ${0.082000 * v1_1_collision_scale}" />
       </geometry>
     </collision>
@@ -575,5 +576,5 @@
       <origin xyz="0.020000 0 0" rpy="0 0 0" />
       <geometry>
-        <box size="0.070000 0.070000 0.070000" />
+        <box size="${0.070000 * v1_1_collision_scale} ${0.070000 * v1_1_collision_scale} ${0.070000 * v1_1_collision_scale}" />
       </geometry>
     </collision>

File: src/my_robot_description/urdf/my_robot.urdf.xacro (robot description, xacro)
@@ -8,4 +8,5 @@
   <xacro:arg name="gravity_compensation_mode" default="off"/>
   <xacro:arg name="gravity_effort_scale" default="0.0"/>
+  <xacro:arg name="j2j3_j3_gravity_effort_scale" default="1.0"/>
   <xacro:arg name="active_real_joints" default=""/>
   <xacro:arg name="can0_interface" default="can0"/>
@@ -26,4 +27,5 @@
     gravity_compensation_mode="$(arg gravity_compensation_mode)"
     gravity_effort_scale="$(arg gravity_effort_scale)"
+    j2j3_j3_gravity_effort_scale="$(arg j2j3_j3_gravity_effort_scale)"
     active_real_joints="$(arg active_real_joints)"
     can0_interface="$(arg can0_interface)"

Commit message: 增加辨识重力补偿工具

File: src/arm_description/urdf/arm.ros2_control.xacro (robot description, xacro)
@@ -1,5 +1,5 @@
 <?xml version="1.0"?>
 <robot xmlns:xacro="http://www.ros.org/wiki/xacro">
-  <xacro:macro name="arm_ros2_control" params="name arm_version:=v1_0 use_mock_hardware:=false gravity_compensation_mode:=off gravity_effort_scale:=0.0 j2j3_j3_gravity_effort_scale:=1.0 active_real_joints:='' can0_interface:=can0 can1_interface:=can1 robot_description_file:=/tmp/robot_description.urdf">
+  <xacro:macro name="arm_ros2_control" params="name arm_version:=v1_0 use_mock_hardware:=false gravity_compensation_mode:=off gravity_effort_scale:=0.0 j2j3_up_poly_a3:=0.0 j2j3_up_poly_a2:=0.0 j2j3_up_poly_a1:=0.0 j2j3_up_poly_a0:=0.0 j2j3_down_poly_a3:=0.0 j2j3_down_poly_a2:=0.0 j2j3_down_poly_a1:=0.0 j2j3_down_poly_a0:=0.0 j2j3_direction_deadband:=0.02 j2j3_direction_smoothing:=0.02 j2j3_j3_gravity_effort_scale:=1.0 active_real_joints:='' can0_interface:=can0 can1_interface:=can1 robot_description_file:=/tmp/robot_description.urdf">
     <xacro:property name="is_arm_v1_1" value="${arm_version == 'v1_1' or arm_version == 'v1.1' or arm_version == '1.1' or arm_version == 1.1}"/>
     <ros2_control name="${name}" type="system">
@@ -15,12 +15,14 @@
         <param name="gravity_effort_scale">${gravity_effort_scale}</param>
         <param name="active_real_joints">${active_real_joints}</param>
-        <param name="j2j3_coupling">0.986</param>
-        <param name="j2j3_j3_scale">1.0</param>
-        <param name="j2j3_j3_offset">0.0</param>
-        <param name="j2j3_poly_a3">0.0</param>
-        <param name="j2j3_poly_a2">0.0</param>
-        <param name="j2j3_poly_a1">0.0</param>
-        <param name="j2j3_poly_a0">0.0</param>
-        <param name="j2j3_scale_mode">divide</param>
+        <param name="j2j3_up_poly_a3">${j2j3_up_poly_a3}</param>
+        <param name="j2j3_up_poly_a2">${j2j3_up_poly_a2}</param>
+        <param name="j2j3_up_poly_a1">${j2j3_up_poly_a1}</param>
+        <param name="j2j3_up_poly_a0">${j2j3_up_poly_a0}</param>
+        <param name="j2j3_down_poly_a3">${j2j3_down_poly_a3}</param>
+        <param name="j2j3_down_poly_a2">${j2j3_down_poly_a2}</param>
+        <param name="j2j3_down_poly_a1">${j2j3_down_poly_a1}</param>
+        <param name="j2j3_down_poly_a0">${j2j3_down_poly_a0}</param>
+        <param name="j2j3_direction_deadband">${j2j3_direction_deadband}</param>
+        <param name="j2j3_direction_smoothing">${j2j3_direction_smoothing}</param>
         <param name="j2j3_j3_gravity_effort_scale">${j2j3_j3_gravity_effort_scale}</param>
       </hardware>
@@ -148,6 +150,6 @@
         <param name="kp">60.0</param>
         <param name="kd">1.0</param>
-        <param name="lower_limit">0.0</param>
-        <param name="upper_limit">1.2</param>
+        <param name="lower_limit">-1.45</param>
+        <param name="upper_limit">0.0</param>
       </joint>
     </ros2_control>

File: src/my_robot_description/urdf/my_robot.urdf.xacro (robot description, xacro)
@@ -8,4 +8,14 @@
   <xacro:arg name="gravity_compensation_mode" default="off"/>
   <xacro:arg name="gravity_effort_scale" default="0.0"/>
+  <xacro:arg name="j2j3_up_poly_a3" default="0.0"/>
+  <xacro:arg name="j2j3_up_poly_a2" default="0.0"/>
+  <xacro:arg name="j2j3_up_poly_a1" default="0.0"/>
+  <xacro:arg name="j2j3_up_poly_a0" default="0.0"/>
+  <xacro:arg name="j2j3_down_poly_a3" default="0.0"/>
+  <xacro:arg name="j2j3_down_poly_a2" default="0.0"/>
+  <xacro:arg name="j2j3_down_poly_a1" default="0.0"/>
+  <xacro:arg name="j2j3_down_poly_a0" default="0.0"/>
+  <xacro:arg name="j2j3_direction_deadband" default="0.02"/>
+  <xacro:arg name="j2j3_direction_smoothing" default="0.02"/>
   <xacro:arg name="j2j3_j3_gravity_effort_scale" default="1.0"/>
   <xacro:arg name="active_real_joints" default=""/>
@@ -27,4 +37,14 @@
     gravity_compensation_mode="$(arg gravity_compensation_mode)"
     gravity_effort_scale="$(arg gravity_effort_scale)"
+    j2j3_up_poly_a3="$(arg j2j3_up_poly_a3)"
+    j2j3_up_poly_a2="$(arg j2j3_up_poly_a2)"
+    j2j3_up_poly_a1="$(arg j2j3_up_poly_a1)"
+    j2j3_up_poly_a0="$(arg j2j3_up_poly_a0)"
+    j2j3_down_poly_a3="$(arg j2j3_down_poly_a3)"
+    j2j3_down_poly_a2="$(arg j2j3_down_poly_a2)"
+    j2j3_down_poly_a1="$(arg j2j3_down_poly_a1)"
+    j2j3_down_poly_a0="$(arg j2j3_down_poly_a0)"
+    j2j3_direction_deadband="$(arg j2j3_direction_deadband)"
+    j2j3_direction_smoothing="$(arg j2j3_direction_smoothing)"
     j2j3_j3_gravity_effort_scale="$(arg j2j3_j3_gravity_effort_scale)"
     active_real_joints="$(arg active_real_joints)"
