Commit message: ``` feat(arm_hardware): 统一J2/J3映射参数并重构硬件接口
- RealArmHardwareInterface和arm.ros2_control.xacro统一使用j2j3_coupling、
  j2j3_j3_scale、j2j3_j3_offset、j2j3_scale_mode以及j2j3_poly_a0..a3参数
- 参数通过control_gains.yaml经launch传入xacro，最终写入URDF的hardware参数
- 从arm_hardware_interface移除重力补偿、控制状态机等相关功能模块
- 更新CMakeLists.txt移除不必要的依赖包和源文件

fix(can): 优化CAN设备集合的消息处理逻辑

- 在DmDeviceCollection中添加电机时正确维护总线分组映射
- 限制CAN消息读取循环防止阻塞，过滤无效帧长度小于8的数据
- 移除电机方向转换逻辑，统一在硬件接口层处理
- 修改sendCommandsWithGains返回类型为bool并增加输入验证
- 修复批量发送命令时的错误处理机制

refactor(ros2_control): 优化xacro宏参数结构

- 更新arm_ros2_control宏参数，统一使用j2j3_前缀的耦合参数
- 为各关节添加可配置的kp/kd增益参数
- 移除过时的j2j3_direction_deadband等参数
- 简化文档中的启动命令示例
```

File: src/arm_description/urdf/arm.ros2_control.xacro (robot description, xacro)
@@ -1,5 +1,5 @@
 <?xml version="1.0"?>
 <robot xmlns:xacro="http://www.ros.org/wiki/xacro">
-  <xacro:macro name="arm_ros2_control" params="name arm_version:=v1_0 use_mock_hardware:=false gravity_compensation_mode:=off gravity_effort_scale:=0.0 j2j3_up_poly_a3:=0.0 j2j3_up_poly_a2:=0.0 j2j3_up_poly_a1:=0.0 j2j3_up_poly_a0:=0.0 j2j3_down_poly_a3:=0.0 j2j3_down_poly_a2:=0.0 j2j3_down_poly_a1:=0.0 j2j3_down_poly_a0:=0.0 j2j3_direction_deadband:=0.02 j2j3_direction_smoothing:=0.02 j2j3_j3_gravity_effort_scale:=1.0 active_real_joints:='' can0_interface:=can0 can1_interface:=can1 robot_description_file:=/tmp/robot_description.urdf">
+  <xacro:macro name="arm_ros2_control" params="name arm_version:=v1_0 use_mock_hardware:=false gravity_compensation_mode:=off gravity_effort_scale:=0.0 j2j3_coupling:=0.0 j2j3_j3_scale:=1.0 j2j3_j3_offset:=0.0 j2j3_scale_mode:=divide j2j3_poly_a3:=0.0 j2j3_poly_a2:=0.0 j2j3_poly_a1:=0.0 j2j3_poly_a0:=0.0 joint1_kp:=120.0 joint1_kd:=3.0 joint2_kp:=240.0 joint2_kd:=3.0 joint3_kp:=240.0 joint3_kd:=3.0 joint4_kp:=120.0 joint4_kd:=3.0 joint5_kp:=120.0 joint5_kd:=3.0 joint6_kp:=120.0 joint6_kd:=1.0 joint7_kp:=60.0 joint7_kd:=1.0 joint_right_finger_kp:=60.0 joint_right_finger_kd:=1.0 active_real_joints:='' can0_interface:=can0 can1_interface:=can1 robot_description_file:=/tmp/robot_description.urdf">
     <xacro:property name="is_arm_v1_1" value="${arm_version == 'v1_1' or arm_version == 'v1.1' or arm_version == '1.1' or arm_version == 1.1}"/>
     <ros2_control name="${name}" type="system">
@@ -15,15 +15,12 @@
         <param name="gravity_effort_scale">${gravity_effort_scale}</param>
         <param name="active_real_joints">${active_real_joints}</param>
-        <param name="j2j3_up_poly_a3">${j2j3_up_poly_a3}</param>
-        <param name="j2j3_up_poly_a2">${j2j3_up_poly_a2}</param>
-        <param name="j2j3_up_poly_a1">${j2j3_up_poly_a1}</param>
-        <param name="j2j3_up_poly_a0">${j2j3_up_poly_a0}</param>
-        <param name="j2j3_down_poly_a3">${j2j3_down_poly_a3}</param>
-        <param name="j2j3_down_poly_a2">${j2j3_down_poly_a2}</param>
-        <param name="j2j3_down_poly_a1">${j2j3_down_poly_a1}</param>
-        <param name="j2j3_down_poly_a0">${j2j3_down_poly_a0}</param>
-        <param name="j2j3_direction_deadband">${j2j3_direction_deadband}</param>
-        <param name="j2j3_direction_smoothing">${j2j3_direction_smoothing}</param>
-        <param name="j2j3_j3_gravity_effort_scale">${j2j3_j3_gravity_effort_scale}</param>
+        <param name="j2j3_coupling">${j2j3_coupling}</param>
+        <param name="j2j3_j3_scale">${j2j3_j3_scale}</param>
+        <param name="j2j3_j3_offset">${j2j3_j3_offset}</param>
+        <param name="j2j3_scale_mode">${j2j3_scale_mode}</param>
+        <param name="j2j3_poly_a3">${j2j3_poly_a3}</param>
+        <param name="j2j3_poly_a2">${j2j3_poly_a2}</param>
+        <param name="j2j3_poly_a1">${j2j3_poly_a1}</param>
+        <param name="j2j3_poly_a0">${j2j3_poly_a0}</param>
       </hardware>
       <!-- J1-J4 使用 CAN 总线 can0 -->
@@ -39,6 +36,6 @@
         <param name="motor_model">J8009</param>
         <param name="can_bus">${can0_interface}</param>
-        <param name="kp">120.0</param>
-        <param name="kd">3.0</param>
+        <param name="kp">${joint1_kp}</param>
+        <param name="kd">${joint1_kd}</param>
         <param name="lower_limit">-2.3562</param>
         <param name="upper_limit">2.3562</param>
@@ -55,6 +52,6 @@
         <param name="motor_model">J8009</param>
         <param name="can_bus">${can0_interface}</param>
-        <param name="kp">240.0</param>
-        <param name="kd">3.0</param>
+        <param name="kp">${joint2_kp}</param>
+        <param name="kd">${joint2_kd}</param>
         <param name="lower_limit">${-0.262 if is_arm_v1_1 else -0.262}</param>
         <param name="upper_limit">${1.204 if is_arm_v1_1 else 1.134}</param>
@@ -70,6 +67,6 @@
         <param name="motor_model">J8009</param>
         <param name="can_bus">${can0_interface}</param>
-        <param name="kp">240.0</param>
-        <param name="kd">3.0</param>
+        <param name="kp">${joint3_kp}</param>
+        <param name="kd">${joint3_kd}</param>
         <param name="lower_limit">-0.9599</param>
         <param name="upper_limit">${1.221 if is_arm_v1_1 else 0.9599}</param>
@@ -85,6 +82,6 @@
         <param name="motor_model">J4340</param>
         <param name="can_bus">${can0_interface}</param>
-        <param name="kp">120.0</param>
-        <param name="kd">3.0</param>
+        <param name="kp">${joint4_kp}</param>
+        <param name="kd">${joint4_kd}</param>
         <param name="lower_limit">${-3.1416 if is_arm_v1_1 else -2.3562}</param>
         <param name="upper_limit">${3.1416 if is_arm_v1_1 else 2.3562}</param>
@@ -101,6 +98,6 @@
         <param name="motor_model">J4340</param>
         <param name="can_bus">${can1_interface}</param>
-        <param name="kp">120.0</param>
-        <param name="kd">3.0</param>
+        <param name="kp">${joint5_kp}</param>
+        <param name="kd">${joint5_kd}</param>
         <param name="lower_limit">${-0.78 if is_arm_v1_1 else -1.5708}</param>
         <param name="upper_limit">1.5708</param>
@@ -117,6 +114,6 @@
         <param name="motor_model">J4310</param>
         <param name="can_bus">${can1_interface}</param>
-        <param name="kp">120.0</param>
-        <param name="kd">1.0</param>
+        <param name="kp">${joint6_kp}</param>
+        <param name="kd">${joint6_kd}</param>
         <param name="lower_limit">-1.5708</param>
         <param name="upper_limit">1.5708</param>
@@ -132,6 +129,6 @@
         <param name="motor_model">J4310</param>
         <param name="can_bus">${can1_interface}</param>
-        <param name="kp">60.0</param>
-        <param name="kd">1.0</param>
+        <param name="kp">${joint7_kp}</param>
+        <param name="kd">${joint7_kd}</param>
         <param name="lower_limit">${-3.1416 if is_arm_v1_1 else -1.5708}</param>
         <param name="upper_limit">${3.1416 if is_arm_v1_1 else 1.5708}</param>
@@ -148,6 +145,6 @@
         <param name="motor_model">J4310</param>
         <param name="can_bus">${can1_interface}</param>
-        <param name="kp">60.0</param>
-        <param name="kd">1.0</param>
+        <param name="kp">${joint_right_finger_kp}</param>
+        <param name="kd">${joint_right_finger_kd}</param>
         <param name="lower_limit">-1.45</param>
         <param name="upper_limit">0.0</param>

File: src/my_robot_description/urdf/my_robot.urdf.xacro (robot description, xacro)
@@ -8,15 +8,28 @@
   <xacro:arg name="gravity_compensation_mode" default="off"/>
   <xacro:arg name="gravity_effort_scale" default="0.0"/>
-  <xacro:arg name="j2j3_up_poly_a3" default="0.0"/>
-  <xacro:arg name="j2j3_up_poly_a2" default="0.0"/>
-  <xacro:arg name="j2j3_up_poly_a1" default="0.0"/>
-  <xacro:arg name="j2j3_up_poly_a0" default="0.0"/>
-  <xacro:arg name="j2j3_down_poly_a3" default="0.0"/>
-  <xacro:arg name="j2j3_down_poly_a2" default="0.0"/>
-  <xacro:arg name="j2j3_down_poly_a1" default="0.0"/>
-  <xacro:arg name="j2j3_down_poly_a0" default="0.0"/>
-  <xacro:arg name="j2j3_direction_deadband" default="0.02"/>
-  <xacro:arg name="j2j3_direction_smoothing" default="0.02"/>
-  <xacro:arg name="j2j3_j3_gravity_effort_scale" default="1.0"/>
+  <xacro:arg name="j2j3_coupling" default="0.0"/>
+  <xacro:arg name="j2j3_j3_scale" default="1.0"/>
+  <xacro:arg name="j2j3_j3_offset" default="0.0"/>
+  <xacro:arg name="j2j3_scale_mode" default="divide"/>
+  <xacro:arg name="j2j3_poly_a3" default="0.0"/>
+  <xacro:arg name="j2j3_poly_a2" default="0.0"/>
+  <xacro:arg name="j2j3_poly_a1" default="0.0"/>
+  <xacro:arg name="j2j3_poly_a0" default="0.0"/>
+  <xacro:arg name="joint1_kp" default="120.0"/>
+  <xacro:arg name="joint1_kd" default="3.0"/>
+  <xacro:arg name="joint2_kp" default="240.0"/>
+  <xacro:arg name="joint2_kd" default="3.0"/>
+  <xacro:arg name="joint3_kp" default="240.0"/>
+  <xacro:arg name="joint3_kd" default="3.0"/>
+  <xacro:arg name="joint4_kp" default="120.0"/>
+  <xacro:arg name="joint4_kd" default="3.0"/>
+  <xacro:arg name="joint5_kp" default="120.0"/>
+  <xacro:arg name="joint5_kd" default="3.0"/>
+  <xacro:arg name="joint6_kp" default="120.0"/>
+  <xacro:arg name="joint6_kd" default="1.0"/>
+  <xacro:arg name="joint7_kp" default="60.0"/>
+  <xacro:arg name="joint7_kd" default="1.0"/>
+  <xacro:arg name="joint_right_finger_kp" default="60.0"/>
+  <xacro:arg name="joint_right_finger_kd" default="1.0"/>
   <xacro:arg name="active_real_joints" default=""/>
   <xacro:arg name="can0_interface" default="can0"/>
@@ -37,15 +50,20 @@
     gravity_compensation_mode="$(arg gravity_compensation_mode)"
     gravity_effort_scale="$(arg gravity_effort_scale)"
-    j2j3_up_poly_a3="$(arg j2j3_up_poly_a3)"
-    j2j3_up_poly_a2="$(arg j2j3_up_poly_a2)"
-    j2j3_up_poly_a1="$(arg j2j3_up_poly_a1)"
-    j2j3_up_poly_a0="$(arg j2j3_up_poly_a0)"
-    j2j3_down_poly_a3="$(arg j2j3_down_poly_a3)"
-    j2j3_down_poly_a2="$(arg j2j3_down_poly_a2)"
-    j2j3_down_poly_a1="$(arg j2j3_down_poly_a1)"
-    j2j3_down_poly_a0="$(arg j2j3_down_poly_a0)"
-    j2j3_direction_deadband="$(arg j2j3_direction_deadband)"
-    j2j3_direction_smoothing="$(arg j2j3_direction_smoothing)"
-    j2j3_j3_gravity_effort_scale="$(arg j2j3_j3_gravity_effort_scale)"
+    j2j3_coupling="$(arg j2j3_coupling)"
+    j2j3_j3_scale="$(arg j2j3_j3_scale)"
+    j2j3_j3_offset="$(arg j2j3_j3_offset)"
+    j2j3_scale_mode="$(arg j2j3_scale_mode)"
+    j2j3_poly_a3="$(arg j2j3_poly_a3)"
+    j2j3_poly_a2="$(arg j2j3_poly_a2)"
+    j2j3_poly_a1="$(arg j2j3_poly_a1)"
+    j2j3_poly_a0="$(arg j2j3_poly_a0)"
+    joint1_kp="$(arg joint1_kp)" joint1_kd="$(arg joint1_kd)"
+    joint2_kp="$(arg joint2_kp)" joint2_kd="$(arg joint2_kd)"
+    joint3_kp="$(arg joint3_kp)" joint3_kd="$(arg joint3_kd)"
+    joint4_kp="$(arg joint4_kp)" joint4_kd="$(arg joint4_kd)"
+    joint5_kp="$(arg joint5_kp)" joint5_kd="$(arg joint5_kd)"
+    joint6_kp="$(arg joint6_kp)" joint6_kd="$(arg joint6_kd)"
+    joint7_kp="$(arg joint7_kp)" joint7_kd="$(arg joint7_kd)"
+    joint_right_finger_kp="$(arg joint_right_finger_kp)" joint_right_finger_kd="$(arg joint_right_finger_kd)"
     active_real_joints="$(arg active_real_joints)"
     can0_interface="$(arg can0_interface)"

Commit message: feat(arm_hardware_interface): 添加MuJoCo硬件接口支持
- 在ros2_control xacro宏中添加use_mujoco_hardware和mujoco_model_path参数
- 实现MujocoArmHardwareInterface插件并添加到CMakeLists.txt
- 在启动文件中添加相应的启动参数配置
- 修改mock硬件接口以添加电机使能发布功能
- 更新URDF文件以支持新的硬件接口参数

refactor(mock_hardware): 优化模拟硬件接口实现

- 在MockArmHardwareInterface中添加enable状态发布
- 持续发布电机使能状态以确保遥控器可以正常控制
- 调整commander的速度参数以适应实际控制需求

File: src/arm_description/urdf/arm.ros2_control.xacro (robot description, xacro)
@@ -1,15 +1,19 @@
 <?xml version="1.0"?>
 <robot xmlns:xacro="http://www.ros.org/wiki/xacro">
-  <xacro:macro name="arm_ros2_control" params="name arm_version:=v1_0 use_mock_hardware:=false gravity_compensation_mode:=off gravity_effort_scale:=0.0 j2j3_coupling:=0.0 j2j3_j3_scale:=1.0 j2j3_j3_offset:=0.0 j2j3_scale_mode:=divide j2j3_poly_a3:=0.0 j2j3_poly_a2:=0.0 j2j3_poly_a1:=0.0 j2j3_poly_a0:=0.0 joint1_kp:=120.0 joint1_kd:=3.0 joint2_kp:=240.0 joint2_kd:=3.0 joint3_kp:=240.0 joint3_kd:=3.0 joint4_kp:=120.0 joint4_kd:=3.0 joint5_kp:=120.0 joint5_kd:=3.0 joint6_kp:=120.0 joint6_kd:=1.0 joint7_kp:=60.0 joint7_kd:=1.0 joint_right_finger_kp:=60.0 joint_right_finger_kd:=1.0 active_real_joints:='' can0_interface:=can0 can1_interface:=can1 robot_description_file:=/tmp/robot_description.urdf">
+  <xacro:macro name="arm_ros2_control" params="name arm_version:=v1_0 use_mock_hardware:=false use_mujoco_hardware:=false mujoco_model_path:='' gravity_compensation_mode:=off gravity_effort_scale:=0.0 j2j3_coupling:=0.0 j2j3_j3_scale:=1.0 j2j3_j3_offset:=0.0 j2j3_scale_mode:=divide j2j3_poly_a3:=0.0 j2j3_poly_a2:=0.0 j2j3_poly_a1:=0.0 j2j3_poly_a0:=0.0 joint1_kp:=120.0 joint1_kd:=3.0 joint2_kp:=240.0 joint2_kd:=3.0 joint3_kp:=240.0 joint3_kd:=3.0 joint4_kp:=120.0 joint4_kd:=3.0 joint5_kp:=120.0 joint5_kd:=3.0 joint6_kp:=120.0 joint6_kd:=1.0 joint7_kp:=60.0 joint7_kd:=1.0 joint_right_finger_kp:=60.0 joint_right_finger_kd:=1.0 active_real_joints:='' can0_interface:=can0 can1_interface:=can1 robot_description_file:=/tmp/robot_description.urdf">
     <xacro:property name="is_arm_v1_1" value="${arm_version == 'v1_1' or arm_version == 'v1.1' or arm_version == '1.1' or arm_version == 1.1}"/>
     <ros2_control name="${name}" type="system">
       <hardware>
-        <xacro:if value="${use_mock_hardware}">
+        <xacro:if value="${use_mujoco_hardware}">
+          <plugin>arm_hardware_interface/MujocoArmHardwareInterface</plugin>
+        </xacro:if>
+        <xacro:if value="${not use_mujoco_hardware and use_mock_hardware}">
           <plugin>arm_hardware_interface/MockArmHardwareInterface</plugin>
         </xacro:if>
-        <xacro:unless value="${use_mock_hardware}">
+        <xacro:if value="${not use_mujoco_hardware and not use_mock_hardware}">
           <plugin>arm_hardware_interface/RealArmHardwareInterface</plugin>
-        </xacro:unless>
+        </xacro:if>
         <param name="robot_description">${robot_description_file}</param>
+        <param name="mujoco_model_path">${mujoco_model_path}</param>
         <param name="gravity_compensation_mode">${gravity_compensation_mode}</param>
         <param name="gravity_effort_scale">${gravity_effort_scale}</param>

File: src/my_robot_description/urdf/my_robot.urdf.xacro (robot description, xacro)
@@ -6,4 +6,6 @@
   <xacro:arg name="gripper_version" default="v1_0"/>
   <xacro:arg name="use_mock_hardware" default="false"/>
+  <xacro:arg name="use_mujoco_hardware" default="false"/>
+  <xacro:arg name="mujoco_model_path" default=""/>
   <xacro:arg name="gravity_compensation_mode" default="off"/>
   <xacro:arg name="gravity_effort_scale" default="0.0"/>
@@ -48,4 +50,6 @@
     arm_version="$(arg arm_version)"
     use_mock_hardware="$(arg use_mock_hardware)"
+    use_mujoco_hardware="$(arg use_mujoco_hardware)"
+    mujoco_model_path="$(arg mujoco_model_path)"
     gravity_compensation_mode="$(arg gravity_compensation_mode)"
     gravity_effort_scale="$(arg gravity_effort_scale)"
